File: spot/HCT_Device/HCT_Device.kicad_sch (KiCad schematic)
At the start: 151 parts, among them J202 Conn_01x06, J203 Conn_01x04, J204 Conn_01x04, J205 Conn_01x08, J206 Conn_01x03, J207 Conn_01x03, J208 Conn_01x06, J209 Conn_01x04, J211 Conn_01x03, J212 Conn_01x04, P203 TP, P204 TP, P205 TP, P208 TP, P209 TP, P210 TP, Q202 NC, Q203 NC, SW202 SW_Push, SW203 SW_Push, U202 NJM2884U1-33-TE1, U203 ESP32-WROOM-32, U207 MCP6002-xSN, U208 MCP6002-I-MS, U209 RX-8035

Commit message: no message
Parts:
- added J210, J211: Conn_01x03, spot:ZH_B3B-ZR, symbol Connector_Generic:Conn_01x03
Connections:
- net GND1: now also J210.2 (Pin_2), J211.2 (Pin_2)
- net Motor2-IN3: now also J210.1 (Pin_1)
- net Motor2-IN4: now also J210.3 (Pin_3)
- net Touch8: now also J211.3 (Pin_3)
- net Touch9: now also J211.1 (Pin_1)
Other:
- note added: "※改造"
- moved on the sheet: Hole201, Hole202, P208, P210
